Commit message: Changed variable names to camel case.

File: urdf/simple2d_arm.urdf (robot description, URDF)
Before this commit: robot simple_two_axis_robot, 6 links, 5 joints
Joints:
- joint joint2: origin xyz=0 0.05 0.5 rpy=0 0 0 -> xyz=0 0 0.5 rpy=0 0 0

Commit message: Fixed to calculate cameraUpVector

File: urdf/simple2d_arm.urdf (robot description, URDF)
Before this commit: robot simple_two_axis_robot, 6 links, 5 joints
Joints:
- joint joint1: origin xyz=0 0.275 1.2 rpy=0 -1.57 0 -> xyz=0 0.4 1.2 rpy=0 -1.57 0

File: urdf/simple_camera.urdf (robot description, URDF)
Before this commit: robot simple_camera, 3 links, 2 joints
Links:
- removed link world
- added link base_link
Joints:
- joint world_joint: parent world -> base_link
