Commit message: add "IBVS", "eye to hand", "eye in hand" notebook

File: urdf/simple6d_arm_with_force_sensor.urdf (robot description, URDF)
Before this commit: robot simple_six_axis_robot, 10 links, 9 joints
Links:
- link base_link: geometry collision cylinder length=0.8 radius=0.15; visual cylinder length=0.8 radius=0.15
Joints:
- joint joint1: origin xyz=0 0 1.1 rpy=0 0 0 -> xyz=0 0 0.8 rpy=0 0 0

File: urdf/simple6d_arm_with_gripper.urdf (robot description, URDF)
Before this commit: robot simple_six_axis_robot, 11 links, 10 joints
Links:
- link base_link: geometry collision cylinder length=0.8 radius=0.15; visual cylinder length=0.8 radius=0.15
- link gripper_left_link: geometry collision box size=0.05 0.05 0.1; visual box size=0.05 0.05 0.1
- link gripper_right_link: geometry collision box size=0.05 0.05 0.1; visual box size=0.05 0.05 0.1
Joints:
- joint joint1: origin xyz=0 0 1.1 rpy=0 0 0 -> xyz=0 0 0.80 rpy=0 0 0

File: urdf/simple_camera.urdf (robot description, URDF)
Before this commit: robot simple_camera, 3 links, 2 joints
Joints:
- joint camera_target_joint: origin xyz=0.01 0.0 0.0 rpy=0 0 0 -> xyz=0.0 0.0 0.01 rpy=0 0 0
