Commit message: add particle filter localization notebook

File: urdf/simple_two_wheel_car.urdf (robot description, URDF)
Before this commit: robot simple_four_wheel_car, 11 links, 10 joints
Links:
- removed link body_link
- added link base_link, mass 10.0; collision box size=0.3 0.3 0.1; visual box size=0.3 0.3 0.1
- link back_caster_link: geometry collision box size=0.05 0.05 0.05; visual box size=0.05 0.05 0.05
- link front_caster_link: geometry collision box size=0.05 0.05 0.05; visual box size=0.05 0.05 0.05
Joints:
- joint back_caster_joint: parent body_link -> base_link
- joint bottom_sensor_joint: parent body_link -> base_link
- joint bumper_joint: parent body_link -> base_link
- joint front_caster_joint: parent body_link -> base_link
- joint front_sensor_joint: parent body_link -> base_link
- joint front_wheel_joint: parent body_link -> base_link
- joint lidar_joint: parent body_link -> base_link
- joint right_wheel_joint: parent body_link -> base_link
